File: VehicleBattVMonIoT_SMD.sch (EAGLE design)
At the start: 55 parts, among them IC1 LD117AS33TR, J1 CON_HEADER_1X06-SMD-RIGHT-ANG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, M1 ARDUINO-PRO-MINI-3.3V#APC, U1 DC-DC-STEP-DOWN-MP1584, U2 ARDUINO_PRO_MINI, U3 RFM69HCW, X1 BU-SMA-G

Commit message: updated arduino pro mini symbol to allow flood
Parts:
- removed IC1: LD117AS33TR, v-reg:LD117AS33TR
- added C12: 100n, 0805, 25v, rcl:C-EUC0805
- added C13: 1uF, 0805, 25V, rcl:C-EUC0805
- added IC3: (no value), SparkFun-PowerIC:V_REG_LM1117SOT223
- added TP3: TP_1MM_TH", TP_1MM_TH:TP_1MM_TH"
- C10, C3, C9: value (none) -> 1uF, 0805, 25V
- C6: value (none) -> 100n, 0805, 25V
- U2: value ARDUINO_PRO_MINI -> 24AA025E64T-I/OT; device SparkFun-Boards:ARDUINO_PRO_MINI -> Microchip-24AA0:24AA025E64T-I/OT
- renumbered U$1 to U4
Connections:
- net +3V3: now also C12.1, C13.1, IC3.OUT, IC3.OUT@1, TP3.1, U2.VCC; no longer IC1.OUT
- net +5V: now also IC3.IN; no longer IC1.IN, U2.RAW
- net /INT: no longer U2.2
- net BT_BRK: no longer U2.*6
- net BT_RXD: no longer U2.*5
- net BT_STATE: no longer U2.*3
- net BT_TXD: no longer U2.4
- net GND: now also C12.2, C13.2, IC3.ADJ, M1.GND.3, U2.A0, U2.A1, U2.VSS; no longer IC1.ADJ, U2.GND, U2.GND@2
- net MISO: no longer U2.12
- net MOSI: no longer U2.*11
- net NSS_1: no longer U2.*10
- net NSS_2: no longer U2.*9
- net PER_RST: no longer U2.7
- net RGB_CTRL: no longer U2.8
- net SCK: no longer U2.13
- net SCL: now also U2.SCL; no longer U2.A5
- net SDA: now also U2.SDA; no longer U2.A4
Other:
- note added: "NC"
- moved on the sheet: TP1, TP2

Commit message: CAD A release for manufacture
Released for manufacture at OSH park
Parts:
- removed SV2: (no value), con-lstb:MA10-1W
- removed U2: 24AA025E64T-I/OT, Microchip-24AA0:24AA025E64T-I/OT
- added IC1: 24AA02E64, microchip:24AA00OT
- added TP4, TP5, TP6, TP7, TP8: TP_1MM_TH", TP_1MM_TH:TP_1MM_TH"
- C11, C2, C7: value (none) -> 1uF, 0805, 25V
- C12: value 100n, 0805, 25v -> 1u, 0805, 25v
- C6: value 100n, 0805, 25V -> 1u, 0805, 25V
- C8: value (none) -> 1n, 0805, 16v
- R4, R6, R7: value 4k7 -> 10k
- SV1: value NOFIT -> (none)
Connections:
- new net ARD_A0: M1.A0, TP4.1
- net +3V3: now also IC1.VCC; no longer SV2.1, U2.VCC
- net ADC_A0: now also TP8.1; no longer SV2.7
- net ADC_A1: now also TP5.1; no longer SV2.8
- net ADC_A2: now also TP6.1; no longer SV2.9
- net ADC_A3: now also TP7.1; no longer SV2.10
- net ALERT: no longer SV2.6
- net GND: now also IC1.GND; no longer SV2.2, SV2.5, U2.A0, U2.A1, U2.VSS
- net SCL: now also IC1.SCL, R1.1, SV1.3; no longer R2.1, SV1.4, SV2.3, U2.SCL
- net SDA: now also IC1.SDA, R2.1, SV1.4; no longer R1.1, SV1.3, SV2.4, U2.SDA
Other:
- note added: "1K CURRENT LIMIT IN CASE OF LEAKAGE FROM 5V INTO 3.3V DOMAIN. REMOVE IF NOT REQUIRED."
- note added: "ADAFRUIT PINOUT I2C ADDR: 0X48 DEFAULT 7BIT"
- note added: "ADS1115 16 BIT ADC FIT ONE ONLY GAIN ERROR AND GAIN DRIFT ARE VERY LOW SO NO NEED FOR A REFERENCE VOLTAGE"
- note added: "ARDUINO PRO MINI 3.3V 8MHz VERSION REQUIRES EXTERNAL USB TO SERIAL CONVERTER **WARNING**: ENSURE EXTERNAL PROGRAMMER IS 3.3V VERSION THE 5V VERSION MAY DAMAGE CIRCUIT"
- note added: "EUI-64 LORA NODE IDENTITY FIT IF EUI NUMBER NOT AVAILABLE ELSEWHERE."
- note added: "NOT ALL WILL BE NEEDED - TBD"
- note added: "OLED I2C MODULE DEBUG USE VIN: 3.3-5V I_IN: P: Full screen lit 0.08W (0.06W typically with screen full of characters) ADDR: 0x3C OR 0x3D 7BIT WRITE 0X78 OR 0X7A 8BIT WRITE SELECTABLE WITH RESISTORS ON OLED"
- note added: "PU MAY BE FITTED ON MODULES"
- note added: "RANGES VIN: 1.7 - 5.5V I_IN: 3MA MAX TEMP: -40 -> +85C I2C ADDR: 0X51 (7BIT WRITE), 0XA0 (8 BIT WRITE) 400k@3.3v 2kPU@400k, 10kPU@100k LOWER NIBBLE EXCEPT R/W ARE DONT CARE"
- note added: "RANGES VIN: IOUT: TEMP:"
- note added: "RGB LED"
- note added: "SHT31 MODULE 2.4 to 5.5 V 0X44 DEFAULT ADAFRUIT (7BIT) OR 0X45 ON OTHERS 1.5MA MAX"
- note added: "SPI FLASH"
- note removed: "ADAFRUIT PINOUT"
- note removed: "ADS1115 16 BIT ADC FIT ONE ONLY SOME BOARDS SWAP SCL/SDA GAIN ERROR AND GAIN DRIFT ARE VERY LOW SO NO NEED FOR A REFERENCE VOLTAGE"
- note removed: "ALTERNATIVE PINOUT"
- note removed: "ARDUINO PRO MINI 3.3V 8MHz VERSION REQUIRES EXTERNAL USB TO SERIAL CONVERTER"
- note removed: "OLED I2C MODULE"
- note removed: "SHT31 MODULE"
- moved on the sheet: C12, C3, TP2
