File: CADB/VehicleBattVMonIoT_SMD.sch (EAGLE design)
At the start: 62 parts, among them IC1 24AA02E64, J1 CON_HEADER_1X06-SMD-RIGHT-ANG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, M1 ARDUINO-PRO-MINI-3.3V#APC, U1 DC-DC-STEP-DOWN-MP1584, U3 RFM69HCW, U4 SPI_FLASH-X25XXSMD, X1 BU-SMA-G

Commit message: Latest CAD B and re-arrange structure
seperate directory for CADA CADB.
Parts:
- added R12: 10k, 5%, rcl:R-EU_R0805
- added TP9: TP_1MM_TH", TP_1MM_TH:TP_1MM_TH"
- C1, C4, C5: value 100uF, 25V -> 100uF, 25V, 85C; MF (none) -> MULTICOMP; MPN (none) -> MCUMR25V107M8X5; OC_FARNELL (none) -> 1870940
- C10, C11, C13, C2, C3, C7, C9: value 1uF, 0805, 25V -> 1uF, 0805, 25V, X5R; MF (none) -> MULTICOMP; MPN (none) -> MC0805X105K250CT; OC_FARNELL (none) -> 2320832
- C12: value 1u, 0805, 25v -> 1uF, 0805, 25V, X5R; MF (none) -> MULTICOMP; MPN (none) -> MC0805X105K250CT; OC_FARNELL (none) -> 2320832
- C6: value 1u, 0805, 25V -> 1uF, 0805, 25V, X5R; MF (none) -> MULTICOMP; MPN (none) -> MC0805X105K250CT; OC_FARNELL (none) -> 2320832
- C8: value 1n, 0805, 16v -> 1NF, 0805, 16V, X5R; MF (none) -> MULTICOMP; MPN (none) -> MCSH21B102K160CT; OC_FARNELL (none) -> 1856432
- D1: MF (none) -> ON SEMICONDUCTOR; MPN (none) -> MBRA340T3G; OC_FARNELL (none) -> 1431078
- D10, D2, D3, D4, D6: MF (none) -> DIODES INC.; MPN (none) -> B0520LW-7-F; OC_FARNELL (none) -> 1773476
- D11: MF (none) -> MULTICOMP; MPN (none) -> 1N4148WS.; OC_FARNELL (none) -> 1466524
- D5, D7, D8: value MBR0520LT -> NOFIT; MF (none) -> DIODES INC.; MPN (none) -> B0520LW-7-F; OC_FARNELL (none) -> 1773476
- D9: value (none) -> WS2812B; OC_FARNELL (none) -> unknown
- F1: MF (none) -> MULTICOMP; MPN (none) -> MC36219.; OC_FARNELL (none) -> 2366776
- H2, H3, H4, H5, M1, PAD1, PAD2, TP1, TP2, TP3, TP4, TP5, TP6, TP7, TP8, U1: OC_FARNELL (none) -> unknown
- IC1: MPN (none) -> 24AA00T-I/OT
- IC3: value (none) -> LM1117; MF (none) -> STMICROELECTRONICS; MPN (none) -> LD1117S33TR; OC_FARNELL (none) -> 1202826
- J1: value CON_HEADER_1X06-SMD-RIGHT-ANGLED -> HM-10 MODULE; OC_FARNELL (none) -> unknown
- JP1: value (none) -> SHT31 MODULE; OC_FARNELL (none) -> unknown
- JP2: value (none) -> OLED MODULE; OC_FARNELL (none) -> unknown
- L1: MF (none) -> COILCRAFT; MPN (none) -> MSS7341-683MLD; OC_FARNELL (none) -> 2288678
- R1, R2, R6, R7: value 10k -> 10k, 5%; MF (none) -> MULTICOMP; MPN (none) -> MC01W0805510K; OC_FARNELL (none) -> 9333720
- R10, R11: value (none) -> 22k, 1%; MF (none) -> WELWYN; MPN (none) -> WCR0805-22KFI; OC_FARNELL (none) -> 1099809
- R3: value 4k7 -> NOFIT; MF (none) -> MULTICOMP; MPN (none) -> MC01W0805510K; OC_FARNELL (none) -> 9333720
- R4: value 10k -> NOFIT; MF (none) -> MULTICOMP; MPN (none) -> MC01W0805510K; OC_FARNELL (none) -> 9333720
- R5: value 1k -> 1k, 5%; MF (none) -> WELWYN; MPN (none) -> WCR0805-1K0FI; OC_FARNELL (none) -> 1099800
- R8, R9: value (none) -> 100k, 1%; MF (none) -> YAGEO (PHYCOMP); MPN (none) -> RC0805FR-07100KL; OC_FARNELL (none) -> 9237879
- SV1: value (none) -> ADS1115 MODULE
- U3: value RFM69HCW -> RFM9xW; OC_FARNELL (none) -> unknown
- U4: value SPI_FLASH-X25XXSMD -> W25Q80DVSNIG; OC_FARNELL (none) -> unknown
- X1: MF (none) -> AMP - TE CONNECTIVITY; MPN (none) -> 5-1814400-1; OC_FARNELL (none) -> 1248989
Connections:
- net /INT: now also D3.C, D4.C, D5.C, D6.C, D7.C, D8.C, R12.2; no longer D3.A, D4.A, D5.A, D6.A, D7.A, D8.A
- net DIO0: now also D4.A; no longer D4.C
- net DIO1: now also D3.A; no longer D3.C
- net DIO2: now also D6.A; no longer D6.C
- net DIO3: now also D5.A; no longer D5.C
- net DIO4: now also D7.A; no longer D7.C
- net DIO5: now also D8.A; no longer D8.C
- net GND: now also R12.1, TP9.1
Other:
- note added: "1K CURRENT LIMIT IN CASE OF LEAKAGE FROM 5V INTO 3.3V DOMAIN. REMOVE IF NOT REQUIRED. TBD"
- note added: "ADAFRUIT PINOUT BEWARE: SOME CLONE BOARDS HAVE I2C SWAPPED I2C ADDR: 0X48 DEFAULT (7BIT ADDRESSING)"
- note added: "ADS1115 16 BIT ADC GAIN ERROR AND GAIN DRIFT ARE VERY LOW SO NO NEED FOR A REFERENCE VOLTAGE"
- note added: "DEBUG USE VIN: 3.3-5V I_IN: P: Full screen lit 0.08W (0.06W typically with screen full of characters) ADDR: 0x3C OR 0x3D 7BIT WRITE 0X78 OR 0X7A 8BIT WRITE SELECTABLE WITH RESISTORS ON OLED"
- note added: "Digikey: Nichicon UMA1E101MDD1TP 25V, £0.26 each Farnell: Multicomp MCUMR25V107M8X5 £0.21 each"
- note added: "LMIC DRIVER REQUIRES ONLY DIO0, 1, 2. ERROR: IRQ IS NORMALLY LOW GOING HIGH WHEN IRQ SET. HAND WIRED TO: DIO0 -> /INT (D2) DIO1 -> BT_STATE (D3) DIO2 -> BT_BRK (D6)"
- note added: "PULL DOWN NOFIT DUE TO KEEPING RFM95 IN RESET DUE TO LMIC LIBRARY USE OF RESET LINE - SUSPECT INPUT,PU INSTEAD OF DRIVEN OUTPUT."
- note added: "RAW + 5V INTO ARDUINO REGULATOR"
- note added: "RESISTORS SET FOR A 3.3V ADC."
- note added: "REVERSE CURRENT PROTECTION DIODE MAY BE LEAKY, NEEDS CORRECTING"
- note added: "SMA Female Jack Bulkhead Solder PCB Mount 5.08mm Right Angle RF Connector"
- note added: "UNUSED INPUTS CAN BE FLOATED OR PULLED TO VCC, NOT GND."
- note removed: "1K CURRENT LIMIT IN CASE OF LEAKAGE FROM 5V INTO 3.3V DOMAIN. REMOVE IF NOT REQUIRED."
- note removed: "ADAFRUIT PINOUT I2C ADDR: 0X48 DEFAULT 7BIT"
- note removed: "ADS1115 16 BIT ADC FIT ONE ONLY GAIN ERROR AND GAIN DRIFT ARE VERY LOW SO NO NEED FOR A REFERENCE VOLTAGE"
- note removed: "FARNELL, Multicomp: MC36219"
- note removed: "NOT ALL WILL BE NEEDED - TBD"
- note removed: "OLED I2C MODULE DEBUG USE VIN: 3.3-5V I_IN: P: Full screen lit 0.08W (0.06W typically with screen full of characters) ADDR: 0x3C OR 0x3D 7BIT WRITE 0X78 OR 0X7A 8BIT WRITE SELECTABLE WITH RESISTORS ON OLED"
- note removed: "REVERSE CURRENT PROTECTION DIODE"
- note removed: "Rubycon 25ML47MEFC6.3X5"
- note removed: "SHOULD THE OTHER ANALOG INPUTS BE GROUNDED?"
- moved on the sheet: C10, C11, C13, C3, C5, D3, D4, D5, D6, D7, D8, D9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

Commit message: minor updates
Parts:
- removed IC1: 24AA02E64, microchip:24AA00OT
- added U2: MICROCHIP-24AA02E64T_24AA02E64T-I/OT, WeMos-Lora:MICROCHIP-24AA02E64T_24AA02E64T-I/OT
Connections:
- net +3V3: now also U2.VCC; no longer IC1.VCC
- net GND: now also U2.VSS; no longer IC1.GND
- net SCL: now also U2.SCL; no longer IC1.SCL
- net SDA: now also U2.SDA; no longer IC1.SDA
Other:
- note added: "LMIC DRIVER REQUIRES ONLY DIO0, 1, 2. ERROR: IRQ IS NORMALLY LOW GOING HIGH WHEN IRQ SET. HAND WIRED TO: DIO0 -> /INT (D2) DIO1 -> BT_STATE (D3) DIO2 -> BT_BRK (D6) SCHEMATIC NEEDS UPDATING DIO3,4,5 MAY BE USED IN CERTAIN MODES SO MAY AS WELL WIRE IN IF POSSIBLE"
- note added: "REVERSE CURRENT PROTECTION DIODE LEAKY, NEEDS CORRECTING"
- note removed: "LMIC DRIVER REQUIRES ONLY DIO0, 1, 2. ERROR: IRQ IS NORMALLY LOW GOING HIGH WHEN IRQ SET. HAND WIRED TO: DIO0 -> /INT (D2) DIO1 -> BT_STATE (D3) DIO2 -> BT_BRK (D6)"
- note removed: "REVERSE CURRENT PROTECTION DIODE MAY BE LEAKY, NEEDS CORRECTING"
